File: dcdc_breakout/dcdc_breakout.kicad_pcb (KiCad board)
At the start: 2 copper layers, 14.5 x 33 mm, 12 parts, among them J1 G2116, U1 DC_DC_BREAKOUT

Commit message: Adjusted footprints, some more changes
Parts:
- moved U1 0.10 mm to (148.6, 105.2)
Changed lines of the file:
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@@
 (kicad_pcb (version 4) (host pcbnew 4.0.6)
   (general
-    (links 24)
-    (no_connects 24)
+    (links 23)
+    (no_connects 23)
     (area 141.174999 88.674999 155.825001 121.825001)
     (thickness 1.6)
@@
     (mod_text_width 0.15)
     (pad_size 3 2)
-    (pad_drill 1)
+    (pad_drill 1.5)
     (pad_to_mask_clearance 0.2)
     (aux_axis_origin 0 0)
@@
     (add_net VSS)
   )
-  (module dcdc_breakout:DC-DC-BREAKOUT (layer F.Cu)
-    (at 148.5 105.25 90)
-    (fp_text reference U1 (at -13.8 8.575 90) (layer F.SilkS)
-      (effects (font (size 1 1) (thickness 0.15)))
-    )
-    (fp_text value DC_DC_BREAKOUT (at -9 -9 90) (layer F.Fab)
-      (effects (font (size 1 1) (thickness 0.15)))
-    )
-    (fp_line (start 16.5 -7.3) (end -16.5 -7.3) (layer F.SilkS) (width 0.15))
-    (fp_line (start 16.5 7.3) (end 16.5 -7.3) (layer F.SilkS) (width 0.15))
-    (fp_line (start -16.5 7.3) (end 16.5 7.3) (layer F.SilkS) (width 0.15))
-    (fp_line (start -16.5 -7.3) (end -16.5 7.3) (layer F.SilkS) (width 0.15))
-    (pad 1 thru_hole rect (at -14.9 -3.6 90) (size 3 2) (drill 1) (layers *.Cu *.Mask)
-      (net 2 GND))
-    (pad e1 thru_hole rect (at -14.9 -6.1 90) (size 3 2) (drill 1) (layers *.Cu *.Mask))
-    (pad 2 thru_hole rect (at -14.9 6.1 90) (size 3 2) (drill 1) (layers *.Cu *.Mask)
-      (net 1 VSS))
-    (pad 2 thru_hole rect (at -14.9 3.6 90) (size 3 2) (drill 1) (layers *.Cu *.Mask)
-      (net 1 VSS))
-    (pad 3 smd rect (at 17.825 -3.2 90) (size 2.6 1.524) (layers F.Cu F.Paste F.Mask)
-      (net 2 GND))
-    (pad 4 smd rect (at 17.825 3.2 90) (size 2.6 1.524) (layers F.Cu F.Paste F.Mask)
-      (net 3 +5V))
-  )
   (module Capacitors_SMD:C_0603 (layer F.Cu)
     (at 148.5 118.5 180)
@@
     )
   )
+  (module dcdc_breakout:DC-DC-BREAKOUT (layer F.Cu)
+    (at 148.6 105.25 90)
+    (fp_text reference U1 (at -13.8 8.575 90) (layer F.SilkS)
+      (effects (font (size 1 1) (thickness 0.15)))
+    )
+    (fp_text value DC_DC_BREAKOUT (at -9 -9 90) (layer F.Fab)
+      (effects (font (size 1 1) (thickness 0.15)))
+    )
+    (fp_line (start 16.5 -7.3) (end -16.5 -7.3) (layer F.SilkS) (width 0.15))
+    (fp_line (start 16.5 7.3) (end 16.5 -7.3) (layer F.SilkS) (width 0.15))
+    (fp_line (start -16.5 7.3) (end 16.5 7.3) (layer F.SilkS) (width 0.15))
+    (fp_line (start -16.5 -7.3) (end -16.5 7.3) (layer F.SilkS) (width 0.15))
+    (pad 1 thru_hole rect (at -14.9 -3.6 90) (size 3 2) (drill 1.5) (layers *.Cu *.Mask)
+      (net 2 GND))
+    (pad 1 thru_hole rect (at -14.9 -6.1 90) (size 3 2) (drill 1.5) (layers *.Cu *.Mask)
+      (net 2 GND))
+    (pad 2 thru_hole rect (at -14.9 6.1 90) (size 3 2) (drill 1.5) (layers *.Cu *.Mask)
+      (net 1 VSS))
+    (pad 2 thru_hole rect (at -14.9 3.6 90) (size 3 2) (drill 1.5) (layers *.Cu *.Mask)
+      (net 1 VSS))
+  )
   (gr_line (start 141.25 121.75) (end 141.25 88.75) (layer Edge.Cuts) (width 0.15))
