File: dcdc_breakout/dcdc_breakout.sch (KiCad schematic (older format))
At the start: 12 parts, among them J1 G2116, U1 DC_DC_BREAKOUT

Commit message: Adjusted footprints, some more changes
Changed lines of the file:
@@
 Connection ~ 7300 3300
-$Comp
-L +5V #PWR01
-U 1 1 5939FAF7
-P 6750 4350
-F 0 "#PWR01" H 6750 4200 50  0001 C CNN
-F 1 "+5V" H 6750 4490 50  0000 C CNN
-F 2 "" H 6750 4350 50  0001 C CNN
-F 3 "" H 6750 4350 50  0001 C CNN
-	1    6750 4350
-	0    1    1    0
-$EndComp
 $Comp
 L +5V #PWR02
@@
 $EndComp
 $Comp
-L GND #PWR05
-U 1 1 5939FDEB
-P 6750 4250
-F 0 "#PWR05" H 6750 4000 50  0001 C CNN
-F 1 "GND" H 6750 4100 50  0000 C CNN
-F 2 "" H 6750 4250 50  0001 C CNN
-F 3 "" H 6750 4250 50  0001 C CNN
-	1    6750 4250
-	0    -1   -1   0
-$EndComp
-$Comp
